Commit message: added docker rendering

File: AlohaMini1/simulation/src/Aloha/urdf/Aloha.urdf (robot description, URDF)
Before this commit: robot Aloha, 19 links, 18 joints
Links:
- link base_link: geometry collision mesh filename=package://aloha/meshes/base_link.STL; visual mesh filename=package://aloha/meshes/base_link.STL
- link left_base: geometry collision mesh filename=package://aloha/meshes/left_base.STL; visual mesh filename=package://aloha/meshes/left_base.STL
- link left_link1: geometry collision mesh filename=package://aloha/meshes/left_link1.STL; visual mesh filename=package://aloha/meshes/left_link1.STL
- link left_link2: geometry collision mesh filename=package://aloha/meshes/left_link2.STL; visual mesh filename=package://aloha/meshes/left_link2.STL
- link left_link3: geometry collision mesh filename=package://aloha/meshes/left_link3.STL; visual mesh filename=package://aloha/meshes/left_link3.STL
- link left_link4: geometry collision mesh filename=package://aloha/meshes/left_link4.STL; visual mesh filename=package://aloha/meshes/left_link4.STL
- link left_link5: geometry collision mesh filename=package://aloha/meshes/left_link5.STL; visual mesh filename=package://aloha/meshes/left_link5.STL
- link left_link6: geometry collision mesh filename=package://aloha/meshes/left_link6.STL; visual mesh filename=package://aloha/meshes/left_link6.STL
- link right_base: geometry collision mesh filename=package://aloha/meshes/right_base.STL; visual mesh filename=package://aloha/meshes/right_base.STL
- link right_link1: geometry collision mesh filename=package://aloha/meshes/right_link1.STL; visual mesh filename=package://aloha/meshes/right_link1.STL
- link right_link2: geometry collision mesh filename=package://aloha/meshes/right_link2.STL; visual mesh filename=package://aloha/meshes/right_link2.STL
- link right_link3: geometry collision mesh filename=package://aloha/meshes/right_link3.STL; visual mesh filename=package://aloha/meshes/right_link3.STL
- link right_link4: geometry collision mesh filename=package://aloha/meshes/right_link4.STL; visual mesh filename=package://aloha/meshes/right_link4.STL
- link right_link5: geometry collision mesh filename=package://aloha/meshes/right_link5.STL; visual mesh filename=package://aloha/meshes/right_link5.STL
- link right_link6: geometry collision mesh filename=package://aloha/meshes/right_link6.STL; visual mesh filename=package://aloha/meshes/right_link6.STL
- link vertical_link: geometry collision mesh filename=package://aloha/meshes/vertical_link.STL; visual mesh filename=package://aloha/meshes/vertical_link.STL
- link wheel1: geometry collision mesh filename=package://aloha/meshes/wheel1.STL; visual mesh filename=package://aloha/meshes/wheel1.STL
- link wheel2: geometry collision mesh filename=package://aloha/meshes/wheel2.STL; visual mesh filename=package://aloha/meshes/wheel2.STL
- link wheel3: geometry collision mesh filename=package://aloha/meshes/wheel3.STL; visual mesh filename=package://aloha/meshes/wheel3.STL
Joints:
- removed joint left_base
- removed joint right_base
- removed joint wheel1
- removed joint wheel2
- removed joint wheel3
- added joint left_base_joint: type fixed, parent vertical_link, child left_base, origin xyz=0.15726 0.026474 0.68821 rpy=1.5721 0 -0.01193, axis 0 0 0
- added joint right_base_joint: type fixed, parent vertical_link, child right_base, origin xyz=-0.156575640990368 0.0302182544430658 0.688907726663402 rpy=1.5720584644847 0 -0.0119300103453133, axis 0 0 0
- added joint wheel1_joint: type continuous, parent base_link, child wheel1, origin xyz=-0.1538 0.091161 0.0422 rpy=0 0 -2.1099, axis 0 -1 0
- added joint wheel2_joint: type continuous, parent base_link, child wheel2, origin xyz=0.15563 0.087993 0.0422 rpy=0 0 2.086, axis 0 -1 0
- added joint wheel3_joint: type continuous, parent base_link, child wheel3, origin xyz=-0.0020354 -0.17875 0.0422 rpy=0 0 0, axis -0.015476 -0.99988 0
