Commit message: update control for the simulator in gazebo

File: AlohaMini1/simulation/src/Aloha/urdf/Aloha.urdf (robot description, URDF)
Before this commit: robot Aloha, 19 links, 18 joints
Joints:
- joint left_joint1: limit lower=0 upper=0 effort=0 velocity=0 -> lower=-3.14159 upper=3.14159 effort=50.0 velocity=3.0
- joint left_joint2: limit lower=0 upper=0 effort=0 velocity=0 -> lower=-3.14159 upper=3.14159 effort=50.0 velocity=3.0
- joint left_joint3: limit lower=0 upper=0 effort=0 velocity=0 -> lower=-3.14159 upper=3.14159 effort=50.0 velocity=3.0
- joint left_joint4: limit lower=0 upper=0 effort=0 velocity=0 -> lower=-3.14159 upper=3.14159 effort=50.0 velocity=3.0
- joint left_joint5: limit lower=0 upper=0 effort=0 velocity=0 -> lower=-3.14159 upper=3.14159 effort=50.0 velocity=3.0
- joint left_joint6: limit lower=0 upper=0 effort=0 velocity=0 -> lower=-3.14159 upper=3.14159 effort=50.0 velocity=3.0
- joint right_joint1: limit lower=0 upper=0 effort=0 velocity=0 -> lower=-3.14159 upper=3.14159 effort=50.0 velocity=3.0
- joint right_joint2: limit lower=0 upper=0 effort=0 velocity=0 -> lower=-3.14159 upper=3.14159 effort=50.0 velocity=3.0
- joint right_joint3: limit lower=0 upper=0 effort=0 velocity=0 -> lower=-3.14159 upper=3.14159 effort=50.0 velocity=3.0
- joint right_joint4: limit lower=0 upper=0 effort=0 velocity=0 -> lower=-3.14159 upper=3.14159 effort=50.0 velocity=3.0
- joint right_joint5: limit lower=0 upper=0 effort=0 velocity=0 -> lower=-3.14159 upper=3.14159 effort=50.0 velocity=3.0
- joint right_joint6: limit lower=0 upper=0 effort=0 velocity=0 -> lower=-3.14159 upper=3.14159 effort=50.0 velocity=3.0
- joint vertical_move: limit lower=0 upper=0 effort=0 velocity=0 -> lower=0.0 upper=0.20 effort=100.0 velocity=0.5
