Commit message: update wheel-contact model and vertical lift

File: AlohaMini1/simulation/src/Aloha/urdf/aloha_cameras.xacro (robot description, xacro)
@@ -53,7 +53,8 @@
   </xacro:macro>
   <xacro:macro name="aloha_cameras">
-    <!-- CAD-derived provisional lens poses. The chest camera moves with the
-         lift carriage. The high head and rear cameras are fixed to base_link.
-         Replace only these origins after physical extrinsic calibration. -->
+    <!-- CAD-derived provisional lens poses. The fixed head/rear mounts are
+         expressed in the ROS-aligned base frame; the chest mount remains
+         relative to the CAD-aligned lift carriage and composes to face base
+         +X. Replace only these origins after physical extrinsic calibration. -->
     <xacro:aloha_camera
       name="chest"
@@ -64,11 +65,11 @@
       name="head"
       parent="base_link"
-      xyz="0 -0.102 1.064"
-      rpy="0 0.78539816339 -1.57079632679"/>
+      xyz="0.102 0 1.064"
+      rpy="0 0.78539816339 0"/>
     <xacro:aloha_camera
       name="rear"
       parent="base_link"
-      xyz="0 0.155 1.057"
-      rpy="0 0.63429 1.57079632679"/>
+      xyz="-0.155 0 1.057"
+      rpy="0 0.63429 3.14159265359"/>
   </xacro:macro>
 </robot>

File: AlohaMini1/simulation/src/Aloha/urdf/aloha_description.xacro (robot description, xacro)
@@ -6,7 +6,38 @@
      For more information, please see http://wiki.ros.org/sw_urdf_exporter -->
 <robot xmlns:xacro="http://www.ros.org/wiki/xacro">
+  <!-- Use a smooth primitive for wheel contact. The detailed omni-wheel STL
+       remains the visual geometry, but its many roller facets make contact
+       forces discontinuous and can let the wheel spin without moving the
+       chassis. The cylinder axis is rotated from URDF +Z onto the wheel's +Y
+       axle; its local +X remains the high-friction rolling direction used by
+       aloha_gazebo.xacro. -->
+  <xacro:property name="wheel_collision_radius" value="0.0495" />
+  <xacro:property name="wheel_collision_width" value="0.0399" />
+  <xacro:property name="wheel_collision_y_offset" value="0.01577" />
+  <xacro:macro name="omni_wheel_collision">
+    <collision>
+      <origin
+        xyz="0 ${wheel_collision_y_offset} 0"
+        rpy="1.57079632679 0 0" />
+      <geometry>
+        <cylinder
+          radius="${wheel_collision_radius}"
+          length="${wheel_collision_width}" />
+      </geometry>
+    </collision>
+  </xacro:macro>
   <xacro:macro name="aloha_description">
-  <link
-    name="base_link">
+  <!-- ROS-facing mobile-base frame (REP 103): +X is the direction faced by
+       the chest, +Y is robot-left, and +Z is up. The SolidWorks export used
+       -Y as the physical forward direction, so keep its untouched geometry
+       and joint coordinates under a fixed, rotated CAD frame. -->
+  <link name="base_link" />
+  <joint name="base_cad_joint" type="fixed">
+    <origin xyz="0 0 0" rpy="0 0 1.57079632679" />
+    <parent link="base_link" />
+    <child link="base_cad_link" />
+  </joint>
+  <link
+    name="base_cad_link">
     <inertial>
       <origin
@@ -77,13 +108,5 @@
       </material>
     </visual>
-    <collision>
-      <origin
-        xyz="0 0 0"
-        rpy="0 0 0" />
-      <geometry>
-        <mesh
-          filename="package://aloha/meshes/wheel1.STL" />
-      </geometry>
-    </collision>
+    <xacro:omni_wheel_collision />
   </link>
   <joint
@@ -94,5 +117,5 @@
       rpy="0 0 -2.1099" />
     <parent
-      link="base_link" />
+      link="base_cad_link" />
     <child
       link="wheel1" />
@@ -133,13 +156,5 @@
       </material>
     </visual>
-    <collision>
-      <origin
-        xyz="0 0 0"
-        rpy="0 0 0" />
-      <geometry>
-        <mesh
-          filename="package://aloha/meshes/wheel2.STL" />
-      </geometry>
-    </collision>
+    <xacro:omni_wheel_collision />
   </link>
   <joint
@@ -150,5 +165,5 @@
       rpy="0 0 2.086" />
     <parent
-      link="base_link" />
+      link="base_cad_link" />
     <child
       link="wheel2" />
@@ -189,13 +204,5 @@
       </material>
     </visual>
-    <collision>
-      <origin
-        xyz="0 0 0"
-        rpy="0 0 0" />
-      <geometry>
-        <mesh
-          filename="package://aloha/meshes/wheel3.STL" />
-      </geometry>
-    </collision>
+    <xacro:omni_wheel_collision />
   </link>
   <joint
@@ -206,5 +213,5 @@
       rpy="0 0 0" />
     <parent
-      link="base_link" />
+      link="base_cad_link" />
     <child
       link="wheel3" />
@@ -262,14 +269,15 @@
       rpy="0 0 0" />
     <parent
-      link="base_link" />
+      link="base_cad_link" />
     <child
       link="vertical_link" />
     <axis
       xyz="0 1.8801E-05 1" />
-    <!-- PLACEHOLDER limit for the prismatic vertical lift (metres). The export
-         left it zero-width; replace with the measured travel/effort/velocity of
-         the real lift. Nonzero range is required for position control. -->
-    <limit
-      lower="0.0"
+    <!-- The CAD assembly pose is the joint's q=0 reference, not the mechanical
+         bottom. The documented 0.60 m lift travel spans 0.40 m below that CAD
+         pose and 0.20 m above it. Verify the endpoints, effort, and velocity
+         against the assembled hardware during calibration. -->
+    <limit
+      lower="-0.40"
       upper="0.20"
       effort="100.0"

File: AlohaMini1/simulation/src/Aloha/urdf/aloha_gazebo.xacro (robot description, xacro)
@@ -1,21 +1,23 @@
 <?xml version="1.0"?>
 <robot xmlns:xacro="http://www.ros.org/wiki/xacro">
+  <xacro:property name="wheel_rolling_friction" value="5.0" />
+  <xacro:property name="wheel_lateral_friction" value="0.01" />
   <xacro:macro name="aloha_gazebo" params="controllers_file">
     <!-- An omni wheel needs strong rolling-direction traction and low lateral
          resistance to approximate its passive rollers. fdir1 is expressed in
-         each wheel collision's local frame. -->
+         each wheel collision's local frame; +X is the rolling direction. -->
     <gazebo reference="wheel1">
-      <mu1>1.0</mu1>
-      <mu2>0.01</mu2>
+      <mu1>${wheel_rolling_friction}</mu1>
+      <mu2>${wheel_lateral_friction}</mu2>
       <fdir1>1 0 0</fdir1>
     </gazebo>
     <gazebo reference="wheel2">
-      <mu1>1.0</mu1>
-      <mu2>0.01</mu2>
+      <mu1>${wheel_rolling_friction}</mu1>
+      <mu2>${wheel_lateral_friction}</mu2>
       <fdir1>1 0 0</fdir1>
     </gazebo>
     <gazebo reference="wheel3">
-      <mu1>1.0</mu1>
-      <mu2>0.01</mu2>
+      <mu1>${wheel_rolling_friction}</mu1>
+      <mu2>${wheel_lateral_friction}</mu2>
       <fdir1>1 0 0</fdir1>
     </gazebo>

File: AlohaMini1/simulation/src/Aloha/urdf/aloha_ros2_control.xacro (robot description, xacro)
@@ -1,6 +1,9 @@
 <?xml version="1.0"?>
 <robot xmlns:xacro="http://www.ros.org/wiki/xacro">
-  <!-- The command interfaces are the sim/real contract. A future Pi hardware
-       composition can reuse the joint list and select its own hardware plugin. -->
+  <!-- A future Pi hardware composition can reuse the joint names while
+       selecting command interfaces that match the real actuators. The
+       gravity-loaded simulated lift uses effort so DART can raise and hold
+       it; the physical lift currently exposes velocity control and requires
+       homing/calibration before it can implement this position contract. -->
   <xacro:macro name="aloha_ros2_control" params="hardware_plugin">
     <ros2_control name="AlohaMiniSystem" type="system">
@@ -30,5 +33,9 @@
         </joint>
       </xacro:macro>
-      <xacro:position_controlled_joint name="vertical_move"/>
+      <joint name="vertical_move">
+        <command_interface name="effort"/>
+        <state_interface name="position"/>
+        <state_interface name="velocity"/>
+      </joint>
       <xacro:position_controlled_joint name="left_joint1"/>
       <xacro:position_controlled_joint name="left_joint2"/>
