Commit message: update omni wheel drive control

File: AlohaMini1/simulation/src/Aloha/urdf/aloha_description.xacro (robot description, xacro)
@@ -1,8 +1,10 @@
 <?xml version="1.0" encoding="utf-8"?>
-<!-- This URDF was automatically created by SolidWorks to URDF Exporter! Originally created by Stephen Brawner (brawner@gmail.com)
+<!-- Core robot description. This file intentionally contains only portable
+     links, joints, visual/collision geometry, and inertial properties. -->
+<!-- This model was originally created by SolidWorks to URDF Exporter. Originally created by Stephen Brawner (brawner@gmail.com)
      Commit Version: 1.6.0-4-g7f85cfe  Build Version: 1.6.7995.38578
      For more information, please see http://wiki.ros.org/sw_urdf_exporter -->
-<robot
-  name="Aloha">
+<robot xmlns:xacro="http://www.ros.org/wiki/xacro">
+  <xacro:macro name="aloha_description">
   <link
     name="base_link">
@@ -1124,122 +1126,4 @@
       velocity="3.0" />
   </joint>
-  <!-- Manually added (not part of the SolidWorks export): give the three drive
-       wheels real contact friction so the passive base stops creeping across
-       the floor. Gazebo/DART reads mu1 (rolling direction) and mu2 (lateral);
-       together with the <dynamics> damping on each wheel joint this holds the
-       base stationary until a real drive controller is added. -->
-  <gazebo reference="wheel1">
-    <mu1>1.0</mu1>
-    <mu2>1.0</mu2>
-  </gazebo>
-  <gazebo reference="wheel2">
-    <mu1>1.0</mu1>
-    <mu2>1.0</mu2>
-  </gazebo>
-  <gazebo reference="wheel3">
-    <mu1>1.0</mu1>
-    <mu2>1.0</mu2>
-  </gazebo>
-  <!-- ==================================================================== -->
-  <!-- ros2_control: hardware interface for gz_ros2_control (added manually, -->
-  <!-- not part of the SolidWorks export). The three drive wheels use a      -->
-  <!-- velocity command interface; the vertical lift and both 6-DOF arms use -->
-  <!-- a position command interface. With a controller actively holding each -->
-  <!-- joint, the base no longer creeps (the earlier passive-physics drift). -->
-  <!-- ==================================================================== -->
-  <ros2_control name="AlohaMiniSystem" type="system">
-    <hardware>
-      <plugin>gz_ros2_control/GazeboSimSystem</plugin>
-    </hardware>
-    <joint name="wheel1_joint">
-      <command_interface name="velocity"/>
-      <state_interface name="position"/>
-      <state_interface name="velocity"/>
-    </joint>
-    <joint name="wheel2_joint">
-      <command_interface name="velocity"/>
-      <state_interface name="position"/>
-      <state_interface name="velocity"/>
-    </joint>
-    <joint name="wheel3_joint">
-      <command_interface name="velocity"/>
-      <state_interface name="position"/>
-      <state_interface name="velocity"/>
-    </joint>
-    <joint name="vertical_move">
-      <command_interface name="position"/>
-      <state_interface name="position"/>
-      <state_interface name="velocity"/>
-    </joint>
-    <joint name="left_joint1">
-      <command_interface name="position"/>
-      <state_interface name="position"/>
-      <state_interface name="velocity"/>
-    </joint>
-    <joint name="left_joint2">
-      <command_interface name="position"/>
-      <state_interface name="position"/>
-      <state_interface name="velocity"/>
-    </joint>
-    <joint name="left_joint3">
-      <command_interface name="position"/>
-      <state_interface name="position"/>
-      <state_interface name="velocity"/>
-    </joint>
-    <joint name="left_joint4">
-      <command_interface name="position"/>
-      <state_interface name="position"/>
-      <state_interface name="velocity"/>
-    </joint>
-    <joint name="left_joint5">
-      <command_interface name="position"/>
-      <state_interface name="position"/>
-      <state_interface name="velocity"/>
-    </joint>
-    <joint name="left_joint6">
-      <command_interface name="position"/>
-      <state_interface name="position"/>
-      <state_interface name="velocity"/>
-    </joint>
-    <joint name="right_joint1">
-      <command_interface name="position"/>
-      <state_interface name="position"/>
-      <state_interface name="velocity"/>
-    </joint>
-    <joint name="right_joint2">
-      <command_interface name="position"/>
-      <state_interface name="position"/>
-      <state_interface name="velocity"/>
-    </joint>
-    <joint name="right_joint3">
-      <command_interface name="position"/>
-      <state_interface name="position"/>
-      <state_interface name="velocity"/>
-    </joint>
-    <joint name="right_joint4">
-      <command_interface name="position"/>
-      <state_interface name="position"/>
-      <state_interface name="velocity"/>
-    </joint>
-    <joint name="right_joint5">
-      <command_interface name="position"/>
-      <state_interface name="position"/>
-      <state_interface name="velocity"/>
-    </joint>
-    <joint name="right_joint6">
-      <command_interface name="position"/>
-      <state_interface name="position"/>
-      <state_interface name="velocity"/>
-    </joint>
-  </ros2_control>
-  <!-- gz_ros2_control system plugin. It hosts a controller_manager inside the
-       Gazebo process. The __CONTROLLERS_YAML__ token is replaced at launch
-       time with the absolute path to config/controllers.yaml (see
-       gazebo.launch.py), which keeps this URDF portable across machines. -->
-  <gazebo>
-    <plugin filename="gz_ros2_control-system"
-            name="gz_ros2_control::GazeboSimROS2ControlPlugin">
-      <parameters>__CONTROLLERS_YAML__</parameters>
-    </plugin>
-  </gazebo>
+  </xacro:macro>
 </robot>

Commit message: gripper fully open to 0

File: AlohaMini1/simulation/src/Aloha/urdf/aloha_description.xacro (robot description, xacro)
@@ -266,5 +266,5 @@
     type="prismatic">
     <origin
-      xyz="-0.001045 -0.067891 0.064"
+      xyz="-0.001045 -0.0678985204 -0.336"
       rpy="0 0 0" />
     <parent
@@ -274,11 +274,11 @@
     <axis
       xyz="0 1.8801E-05 1" />
-    <!-- The CAD assembly pose is the joint's q=0 reference, not the mechanical
-         bottom. The documented 0.60 m lift travel spans 0.40 m below that CAD
-         pose and 0.20 m above it. Verify the endpoints, effort, and velocity
-         against the assembled hardware during calibration. -->
-    <limit
-      lower="-0.40"
-      upper="0.20"
+    <!-- q is height above the mechanical bottom: q=0 is the bottom and
+         positive motion raises the lift. Moving this joint origin 0.40 m down
+         its axis preserves the exported CAD assembly at q=0.40 m. Verify the
+         usable endpoints, effort, and velocity on assembled hardware. -->
+    <limit
+      lower="0.0"
+      upper="0.60"
       effort="100.0"
       velocity="0.5" />
@@ -699,11 +699,11 @@
     <axis
       xyz="-0.999889727846743 0.0120164296808642 -0.00872568417324989" />
-    <!-- PLACEHOLDER limit: the SolidWorks export left this joint zero-width.
-         Replace lower/upper/effort/velocity with values measured from the real
-         servo before relying on this for anything quantitative. Nonzero limits
-         are required so the position controller can actually move the joint. -->
-    <limit
-      lower="-3.14159"
-      upper="3.14159"
+    <!-- Operator endpoints derived from the CAD jaw geometry are q=0 (open)
+         and q=-1.57 (closed). Keep the simulation hard stops 0.01 rad beyond
+         them so DART does not pin the velocity-backed joint at either endpoint.
+         Replace these limits with calibrated endpoints for real hardware. -->
+    <limit
+      lower="-1.58"
+      upper="0.01"
       effort="50.0"
       velocity="3.0" />
@@ -1124,11 +1124,11 @@
     <axis
       xyz="-0.999889727846743 0.0120164296808642 -0.00872568417324984" />
-    <!-- PLACEHOLDER limit: the SolidWorks export left this joint zero-width.
-         Replace lower/upper/effort/velocity with values measured from the real
-         servo before relying on this for anything quantitative. Nonzero limits
-         are required so the position controller can actually move the joint. -->
-    <limit
-      lower="-3.14159"
-      upper="3.14159"
+    <!-- Operator endpoints derived from the CAD jaw geometry are q=0 (open)
+         and q=-1.57 (closed). Keep the simulation hard stops 0.01 rad beyond
+         them so DART does not pin the velocity-backed joint at either endpoint.
+         Replace these limits with calibrated endpoints for real hardware. -->
+    <limit
+      lower="-1.58"
+      upper="0.01"
       effort="50.0"
       velocity="3.0" />
